File: KiCad/keyboard.kicad_pcb (KiCad board)
At the start: 2 copper layers, 0 parts

Commit message: PCB
Parts:
- added D1: D_Small, chinh4thepro:ComboDiode, F.Cu at (63.6, 108.8)
- added D10: D_Small, chinh4thepro:ComboDiode, F.Cu at (120.6, 112.8)
- added D11: D_Small, chinh4thepro:ComboDiode, F.Cu at (139.6, 119.8)
- added D12: D_Small, chinh4thepro:ComboDiode, F.Cu at (158.6, 121.8)
- added D13: D_Small, chinh4thepro:ComboDiode, F.Cu at (63.6, 146.8)
- added D14: D_Small, chinh4thepro:ComboDiode, F.Cu at (82.6, 146.8)
- added D15: D_Small, chinh4thepro:ComboDiode, F.Cu at (101.6, 136.8)
- added D16: D_Small, chinh4thepro:ComboDiode, F.Cu at (120.6, 131.8)
- added D17: D_Small, chinh4thepro:ComboDiode, F.Cu at (139.6, 138.8)
- added D18: D_Small, chinh4thepro:ComboDiode, F.Cu at (158.6, 140.8)
- added D19: D_Small, chinh4thepro:ComboDiode, F.Cu at (63.6, 165.8)
- added D2: D_Small, chinh4thepro:ComboDiode, F.Cu at (82.6, 108.8)
- added D20: D_Small, chinh4thepro:ComboDiode, F.Cu at (82.6, 165.8)
- added D21: D_Small, chinh4thepro:ComboDiode, F.Cu at (101.6, 155.8)
- added D22: D_Small, chinh4thepro:ComboDiode, F.Cu at (120.6, 150.8)
- added D23: D_Small, chinh4thepro:ComboDiode, F.Cu at (139.6, 157.8)
- added D24: D_Small, chinh4thepro:ComboDiode, F.Cu at (158.6, 159.8)
- added D25: D_Small, chinh4thepro:ComboDiode, F.Cu at (132.2, 192.6)
- added D26: D_Small, chinh4thepro:ComboDiode, F.Cu at (156.8, 187.4)
- added D27: D_Small, chinh4thepro:ComboDiode, F.Cu at (181.4, 192.6)
- added D28: D_Small, chinh4thepro:ComboDiode, F.Cu at (345.6, 108.8)
- added D29: D_Small, chinh4thepro:ComboDiode, F.Cu at (345.6, 127.8)
- added D3: D_Small, chinh4thepro:ComboDiode, F.Cu at (101.6, 98.8)
- added D30: D_Small, chinh4thepro:ComboDiode, F.Cu at (345.6, 146.8)
- added D31: D_Small, chinh4thepro:ComboDiode, F.Cu at (345.6, 165.8)
- added D32: D_Small, chinh4thepro:ComboDiode, F.Cu at (326.6, 108.8)
- added D33: D_Small, chinh4thepro:ComboDiode, F.Cu at (326.6, 127.8)
- added D34: D_Small, chinh4thepro:ComboDiode, F.Cu at (326.6, 146.8)
- added D35: D_Small, chinh4thepro:ComboDiode, F.Cu at (326.6, 165.8)
- added D36: D_Small, chinh4thepro:ComboDiode, F.Cu at (307.6, 98.8)
- added D37: D_Small, chinh4thepro:ComboDiode, F.Cu at (307.6, 117.8)
- added D38: D_Small, chinh4thepro:ComboDiode, F.Cu at (307.6, 136.8)
- added D39: D_Small, chinh4thepro:ComboDiode, F.Cu at (307.6, 155.8)
- added D4: D_Small, chinh4thepro:ComboDiode, F.Cu at (120.6, 93.8)
- added D40: D_Small, chinh4thepro:ComboDiode, F.Cu at (288.6, 93.8)
- added D41: D_Small, chinh4thepro:ComboDiode, F.Cu at (288.6, 112.8)
- added D42: D_Small, chinh4thepro:ComboDiode, F.Cu at (288.6, 131.8)
- added D43: D_Small, chinh4thepro:ComboDiode, F.Cu at (288.6, 150.8)
- added D44: D_Small, chinh4thepro:ComboDiode, F.Cu at (277.0, 192.6)
- added D45: D_Small, chinh4thepro:ComboDiode, F.Cu at (269.6, 100.8)
- added D46: D_Small, chinh4thepro:ComboDiode, F.Cu at (269.6, 119.8)
- added D47: D_Small, chinh4thepro:ComboDiode, F.Cu at (269.6, 138.8)
- added D48: D_Small, chinh4thepro:ComboDiode, F.Cu at (269.6, 157.8)
- added D49: D_Small, chinh4thepro:ComboDiode, F.Cu at (252.4, 187.4)
- added D5: D_Small, chinh4thepro:ComboDiode, F.Cu at (139.6, 100.8)
- added D50: D_Small, chinh4thepro:ComboDiode, F.Cu at (250.6, 102.8)
- added D51: D_Small, chinh4thepro:ComboDiode, F.Cu at (250.6, 121.8)
- added D52: D_Small, chinh4thepro:ComboDiode, F.Cu at (250.6, 140.8)
- added D53: D_Small, chinh4thepro:ComboDiode, F.Cu at (250.6, 159.8)
- added D54: D_Small, chinh4thepro:ComboDiode, F.Cu at (227.8, 192.6)
- added D6: D_Small, chinh4thepro:ComboDiode, F.Cu at (158.6, 102.8)
- added D7: D_Small, chinh4thepro:ComboDiode, F.Cu at (63.6, 127.8)
- added D8: D_Small, chinh4thepro:ComboDiode, F.Cu at (82.6, 127.8)
- added D9: D_Small, chinh4thepro:ComboDiode, F.Cu at (101.6, 117.8)
- added H1: , ceoloide:mounting_hole_plated, F.Cu at (73.1, 113.3)
- added H10: , ceoloide:mounting_hole_plated, F.Cu at (260.1, 145.3)
- added H11: , ceoloide:mounting_hole_plated, F.Cu at (266.6, 182.4)
- added H12: , ceoloide:mounting_hole_plated, F.Cu at (238.1, 182.4)
- added H2: , ceoloide:mounting_hole_plated, F.Cu at (149.1, 107.3)
- added H3: , ceoloide:mounting_hole_plated, F.Cu at (73.1, 151.3)
- added H4: , ceoloide:mounting_hole_plated, F.Cu at (149.1, 145.3)
- added H5: , ceoloide:mounting_hole_plated, F.Cu at (142.6, 182.4)
- added H6: , ceoloide:mounting_hole_plated, F.Cu at (171.1, 182.4)
- added H7: , ceoloide:mounting_hole_plated, F.Cu at (336.1, 113.3)
- added H8: , ceoloide:mounting_hole_plated, F.Cu at (260.1, 107.3)
- added H9: , ceoloide:mounting_hole_plated, F.Cu at (336.1, 151.3)
- added J1: OLED_128x32, ScottoKeebs_Components:OLED_128x32, F.Cu at (184.6, 105.4)
- added J2: Conn_01x02_Socket, Connector_JST:JST_PH_S2B-PH-K_1x02_P2.00mm_Horizontal, B.Cu at (193.8, 102.3)
- added J3: 4P4C, Connector_RJ:RJ9_Evercom_5301-440xxx_Horizontal, F.Cu at (197.0, 97.0)
- added J4: OLED_128x32, ScottoKeebs_Components:OLED_128x32, F.Cu at (236.6, 105.4)
- added J5: Conn_01x02_Socket, Connector_JST:JST_PH_S2B-PH-K_1x02_P2.00mm_Horizontal, B.Cu at (217.4, 102.5)
- added J6: 4P4C, Connector_RJ:RJ9_Evercom_5301-440xxx_Horizontal, F.Cu at (215.9, 97.0)
- added S1: Keyswitch, ScottoKeebs_Hotswap:Hotswap_MX, F.Cu at (63.6, 103.8)
- added S10: Keyswitch, ScottoKeebs_Hotswap:Hotswap_MX, F.Cu at (120.6, 107.8)
- added S11: Keyswitch, ScottoKeebs_Hotswap:Hotswap_MX, F.Cu at (139.6, 114.8)
- added S12: Keyswitch, ScottoKeebs_Hotswap:Hotswap_MX, F.Cu at (158.6, 116.8)
- added S13: Keyswitch, ScottoKeebs_Hotswap:Hotswap_MX, F.Cu at (63.6, 141.8)
- added S14: Keyswitch, ScottoKeebs_Hotswap:Hotswap_MX, F.Cu at (82.6, 141.8)
- added S15: Keyswitch, ScottoKeebs_Hotswap:Hotswap_MX, F.Cu at (101.6, 131.8)
- added S16: Keyswitch, ScottoKeebs_Hotswap:Hotswap_MX, F.Cu at (120.6, 126.8)
- added S17: Keyswitch, ScottoKeebs_Hotswap:Hotswap_MX, F.Cu at (139.6, 133.8)
- added S18: Keyswitch, ScottoKeebs_Hotswap:Hotswap_MX, F.Cu at (158.6, 135.8)
- added S19: Keyswitch, ScottoKeebs_Hotswap:Hotswap_MX, F.Cu at (63.6, 160.8)
- added S2: Keyswitch, ScottoKeebs_Hotswap:Hotswap_MX, F.Cu at (82.6, 103.8)
- added S20: Keyswitch, ScottoKeebs_Hotswap:Hotswap_MX, F.Cu at (82.6, 160.8)
- added S21: Keyswitch, ScottoKeebs_Hotswap:Hotswap_MX, F.Cu at (101.6, 150.8)
- added S22: Keyswitch, ScottoKeebs_Hotswap:Hotswap_MX, F.Cu at (120.6, 145.8)
- added S23: Keyswitch, ScottoKeebs_Hotswap:Hotswap_MX, F.Cu at (139.6, 152.8)
- added S24: Keyswitch, ScottoKeebs_Hotswap:Hotswap_MX, F.Cu at (158.6, 154.8)
- added S25: Keyswitch, ScottoKeebs_Hotswap:Hotswap_MX, F.Cu at (130.1, 188.0)
- added S26: Keyswitch, ScottoKeebs_Hotswap:Hotswap_MX, F.Cu at (156.8, 182.4)
- added S27: Keyswitch, ScottoKeebs_Hotswap:Hotswap_MX, F.Cu at (183.5, 188.0)
- added S28: Keyswitch, ScottoKeebs_Hotswap:Hotswap_MX, F.Cu at (345.6, 103.8)
- added S29: Keyswitch, ScottoKeebs_Hotswap:Hotswap_MX, F.Cu at (345.6, 122.8)
- added S3: Keyswitch, ScottoKeebs_Hotswap:Hotswap_MX, F.Cu at (101.6, 93.8)
- added S30: Keyswitch, ScottoKeebs_Hotswap:Hotswap_MX, F.Cu at (345.6, 141.8)
- added S31: Keyswitch, ScottoKeebs_Hotswap:Hotswap_MX, F.Cu at (345.6, 160.8)
- added S32: Keyswitch, ScottoKeebs_Hotswap:Hotswap_MX, F.Cu at (326.6, 103.8)
- added S33: Keyswitch, ScottoKeebs_Hotswap:Hotswap_MX, F.Cu at (326.6, 122.8)
- added S34: Keyswitch, ScottoKeebs_Hotswap:Hotswap_MX, F.Cu at (326.6, 141.8)
- added S35: Keyswitch, ScottoKeebs_Hotswap:Hotswap_MX, F.Cu at (326.6, 160.8)
- added S36: Keyswitch, ScottoKeebs_Hotswap:Hotswap_MX, F.Cu at (307.6, 93.8)
- added S37: Keyswitch, ScottoKeebs_Hotswap:Hotswap_MX, F.Cu at (307.6, 112.8)
- added S38: Keyswitch, ScottoKeebs_Hotswap:Hotswap_MX, F.Cu at (307.6, 131.8)
- added S39: Keyswitch, ScottoKeebs_Hotswap:Hotswap_MX, F.Cu at (307.6, 150.8)
- added S4: Keyswitch, ScottoKeebs_Hotswap:Hotswap_MX, F.Cu at (120.6, 88.8)
- added S40: Keyswitch, ScottoKeebs_Hotswap:Hotswap_MX, F.Cu at (288.6, 88.8)
- added S41: Keyswitch, ScottoKeebs_Hotswap:Hotswap_MX, F.Cu at (288.6, 107.8)
- added S42: Keyswitch, ScottoKeebs_Hotswap:Hotswap_MX, F.Cu at (288.6, 126.8)
- added S43: Keyswitch, ScottoKeebs_Hotswap:Hotswap_MX, F.Cu at (288.6, 145.8)
- added S44: Keyswitch, ScottoKeebs_Hotswap:Hotswap_MX, F.Cu at (279.1, 188.0)
- added S45: Keyswitch, ScottoKeebs_Hotswap:Hotswap_MX, F.Cu at (269.6, 95.8)
- added S46: Keyswitch, ScottoKeebs_Hotswap:Hotswap_MX, F.Cu at (269.6, 114.8)
- added S47: Keyswitch, ScottoKeebs_Hotswap:Hotswap_MX, F.Cu at (269.6, 133.8)
- added S48: Keyswitch, ScottoKeebs_Hotswap:Hotswap_MX, F.Cu at (269.6, 152.8)
- added S49: Keyswitch, ScottoKeebs_Hotswap:Hotswap_MX, F.Cu at (252.4, 182.4)
- added S5: Keyswitch, ScottoKeebs_Hotswap:Hotswap_MX, F.Cu at (139.6, 95.8)
- added S50: Keyswitch, ScottoKeebs_Hotswap:Hotswap_MX, F.Cu at (250.6, 97.8)
- added S51: Keyswitch, ScottoKeebs_Hotswap:Hotswap_MX, F.Cu at (250.6, 116.8)
- added S52: Keyswitch, ScottoKeebs_Hotswap:Hotswap_MX, F.Cu at (250.6, 135.8)
- added S53: Keyswitch, ScottoKeebs_Hotswap:Hotswap_MX, F.Cu at (250.6, 154.8)
- added S54: Keyswitch, ScottoKeebs_Hotswap:Hotswap_MX, F.Cu at (225.6, 188.0)
- added S6: Keyswitch, ScottoKeebs_Hotswap:Hotswap_MX, F.Cu at (158.6, 97.8)
- added S7: Keyswitch, ScottoKeebs_Hotswap:Hotswap_MX, F.Cu at (63.6, 122.8)
- added S8: Keyswitch, ScottoKeebs_Hotswap:Hotswap_MX, F.Cu at (82.6, 122.8)
- added S9: Keyswitch, ScottoKeebs_Hotswap:Hotswap_MX, F.Cu at (101.6, 112.8)
- added SW1: Switch, chinh4thepro:reset_switch_smd_side, F.Cu at (164.6, 86.2)
- added SW2: SW_SPDT, chinh4thepro:power_switch_smd_side, F.Cu at (154.6, 86.4)
- added SW3: Switch, chinh4thepro:reset_switch_smd_side, F.Cu at (244.6, 86.2)
- added SW4: SW_SPDT, chinh4thepro:power_switch_smd_side, F.Cu at (254.6, 86.4)
- added U1: XIAO-HALF-HOLE-23P, xiao ESP32S3 Plus_PCB:Xiao_ESP32S3_Plus.kicad_sym, F.Cu at (178.5, 94.4)
- added U3: XIAO-HALF-HOLE-23P, xiao ESP32S3 Plus_PCB:Xiao_ESP32S3_Plus.kicad_sym, F.Cu at (230.6, 94.4)
Routing:
- net L_ROW4: track 0.00 -> 243.4 mm
- net R_ROW4: track 0.00 -> 235.7 mm
- net L_ROW3: track 0.00 -> 224.5 mm
- net R_ROW3: track 0.00 -> 217.4 mm
- net R_ROW5: track 0.00 -> 209.1 mm
- net L_ROW2: track 0.00 -> 205.0 mm
- net R_COL1: track 0.00 -> 201.4 mm
- net R_ROW2: track 0.00 -> 200.3 mm
- net L_ROW1: track 0.00 -> 193.7 mm
- net L_COL1: track 0.00 -> 190.3 mm
- net L_ROW5: track 0.00 -> 184.8 mm
- net R_ROW1: track 0.00 -> 184.6 mm
- net L_COL4: track 0.00 -> 171.5 mm
- net L_COL2: track 0.00 -> 171.3 mm
- net R_COL2: track 0.00 -> 163.0 mm
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Other:
- board outline added: 305 x 125.4 mm
