File: KiCad/keyboard.kicad_pcb (KiCad board)
At the start: 2 copper layers, 305 x 125.4 mm, 132 parts, among them J1 OLED_128x32, J2 Conn_01x02_Socket, J3 4P4C, J4 OLED_128x32, J5 Conn_01x02_Socket, J6 4P4C, SW1 Switch, SW2 SW_SPDT, SW3 Switch, SW4 SW_SPDT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

Commit message: mousebites
Parts:
- added mouse-bite-2mm-slot: VAL**, Panelization:mouse-bite-2mm-slot, F.Cu at (290.1, 76.2)
- added mouse-bite-2mm-slot: VAL**, Panelization:mouse-bite-2mm-slot, F.Cu at (121.2, 76.2)
Other:
- board size 305 x 125.4 mm -> 305 x 137.6 mm

Commit message: partially update pt2
Parts:
- J3, J6: footprint Connector_RJ:RJ9_Evercom_5301-440xxx_Horizontal -> chinh4thepro:RJ9_Evercom_5301-440xxx_Horizontal

Commit message: complete images
Parts:
- removed mouse-bite-2mm-slot (x2): VAL**, Panelization:mouse-bite-2mm-slot
- added G***: LOGO, LOGO, F.Cu at (218.3, 161.9)
- added G***: LOGO, LOGO, F.Cu at (177.3, 101.7)
- added G***: LOGO, LOGO, F.Cu at (56.7, 129.3)
- added G***: LOGO, LOGO, F.Cu at (90.2, 131.7)
- added G***: LOGO, LOGO, F.Cu at (141.9, 131.0)
- added G***: LOGO, LOGO, F.Cu at (352.0, 104.0)
- added G***: LOGO, LOGO, B.Cu at (112.1, 136.0)
- added G***: LOGO, LOGO, B.Cu at (85.9, 128.7)
- added G***: LOGO, LOGO, B.Cu at (215.9, 180.9)
- added G***: LOGO, LOGO, B.Cu at (73.0, 162.6)
- added G***: LOGO, LOGO, B.Cu at (291.3, 164.3)
- added G***: LOGO, LOGO, F.Cu at (272.4, 184.2)
- added G***: LOGO, LOGO, B.Cu at (61.9, 130.6)
- added G***: LOGO, LOGO, B.Cu at (311.0, 163.9)
- added G***: LOGO, LOGO, B.Cu at (153.5, 128.7)
- added G***: LOGO, LOGO, B.Cu at (238.7, 116.9)
- added G***: LOGO, LOGO, B.Cu at (118.1, 98.5)
- added G***: LOGO, LOGO, B.Cu at (259.7, 130.2)
- added G***: LOGO, LOGO, B.Cu at (90.4, 108.8)
- added G***: LOGO, LOGO, B.Cu at (169.6, 170.6)
- added G***: LOGO, LOGO, B.Cu at (293.4, 98.5)
- added G***: LOGO, LOGO, B.Cu at (97.7, 141.8)
- added G***: LOGO, LOGO, F.Cu at (263.8, 133.8)
- added G***: LOGO, LOGO, B.Cu at (113.4, 157.9)
- added G***: LOGO, LOGO, B.Cu at (168.7, 118.4)
- added G***: LOGO, LOGO, B.Cu at (130.1, 145.0)
- added G***: LOGO, LOGO, B.Cu at (182.8, 146.4)
- added G***: LOGO, LOGO, B.Cu at (336.3, 102.1)
- added G***: LOGO, LOGO, B.Cu at (267.2, 168.0)
- added G***: LOGO, LOGO, B.Cu at (91.0, 152.5)
- added G***: LOGO, LOGO, B.Cu at (316.0, 122.7)
- added G***: LOGO, LOGO, B.Cu at (240.0, 135.8)
- added G***: LOGO, LOGO, B.Cu at (279.7, 147.8)
- added G***: LOGO, LOGO, F.Cu at (240.8, 183.8)
- added G***: LOGO, LOGO, B.Cu at (73.9, 139.9)
- added G***: LOGO, LOGO, B.Cu at (74.3, 105.8)
- added G***: LOGO, LOGO, B.Cu at (240.2, 169.3)
- added G***: LOGO, LOGO, B.Cu at (126.7, 168.0)
- added G***: LOGO, LOGO, B.Cu at (165.3, 139.4)
- added G***: LOGO, LOGO, B.Cu at (299.4, 86.9)
- added G***: LOGO, LOGO, B.Cu at (269.2, 106.2)
- added G***: LOGO, LOGO, B.Cu at (317.0, 107.7)
- added G***: LOGO, LOGO, B.Cu at (130.3, 125.1)
- added G***: LOGO, LOGO, B.Cu at (99.4, 165.2)
- added G***: LOGO, LOGO, F.Cu at (135.4, 183.0)
- added G***: LOGO, LOGO, B.Cu at (215.1, 114.6)
- added G***: LOGO, LOGO, B.Cu at (299.2, 139.0)
- added G***: LOGO, LOGO, B.Cu at (225.6, 146.2)
- added G***: LOGO, LOGO, B.Cu at (115.1, 176.6)
- added G***: LOGO, LOGO, B.Cu at (196.2, 112.8)
- added G***: LOGO, LOGO, B.Cu at (103.7, 122.1)
- added G***: LOGO, LOGO, B.Cu at (335.7, 140.1)
- added G***: LOGO, LOGO, B.Cu at (144.5, 170.6)
- added G***: LOGO, LOGO, B.Cu at (141.1, 106.2)
- added G***: LOGO, LOGO, B.Cu at (277.8, 120.8)
- added G***: LOGO, LOGO, F.Cu at (318.6, 133.2)
- added G***: LOGO, LOGO, B.Cu at (60.6, 151.9)
- added G***: LOGO, LOGO, B.Cu at (297.5, 117.3)
- added G***: LOGO, LOGO, B.Cu at (149.0, 154.9)
- added G***: LOGO, LOGO, B.Cu at (193.2, 181.1)
- added G***: LOGO, LOGO, B.Cu at (281.2, 176.1)
- added G***: LOGO, LOGO, F.Cu at (188.8, 162.2)
- added G***: LOGO, LOGO, F.Cu at (164.0, 182.1)
- added G***: LOGO, LOGO, F.Cu at (354.1, 162.6)
Routing:
- net GND: track 161.4 -> 157.7 mm
- net L_ROW1: track 193.7 -> 190.0 mm
- net L_COL2: track 171.3 -> 168.0 mm
- net R_COL4: track 150.5 -> 147.3 mm
- net L_ROW3: track 224.5 -> 221.3 mm
- net R_COL5: track 133.9 -> 131.0 mm
- net R_COL2: track 163.0 -> 160.3 mm
- net R_ROW1: track 184.6 -> 181.9 mm
- net L_COL1: track 190.3 -> 187.6 mm
- net R_COL3: track 137.8 -> 135.3 mm
- net L_ROW2: track 205.0 -> 202.5 mm
- net L_RAW: track 92.4 -> 89.9 mm
- net R_RAW: track 74.9 -> 72.8 mm
- net L_COL6: track 135.2 -> 133.4 mm
- net L_COL5: track 140.9 -> 139.2 mm
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Other:
- board size 305 x 137.6 mm -> 305 x 125.4 mm

Commit message: update images
Parts:
- added G***: LOGO, LOGO, F.Cu at (195.6, 123.3)
- added G***: LOGO, LOGO, F.Cu at (212.9, 123.4)

Commit message: redo mousebites cause i forgor
Parts:
- added REF**: mousebites 2mm, PCM_marbastlib-various:mousebites_2mm, F.Cu at (252.6, 193.5)
- added REF**: mousebites 2mm, PCM_marbastlib-various:mousebites_2mm, F.Cu at (156.2, 193.6)
- added REF**: mousebites 2mm, PCM_marbastlib-various:mousebites_2mm, F.Cu at (120.2, 77.2)
- added REF**: mousebites 2mm, PCM_marbastlib-various:mousebites_2mm, F.Cu at (289.0, 77.2)
Other:
- board size 305 x 125.4 mm -> 307.2 x 148.8 mm
