File: CAD/KiCad/keyboard.kicad_pcb (KiCad board)
At the start: 2 copper layers, 307.2 x 148.8 mm, 202 parts, among them J1 OLED_128x32, J2 Conn_01x02_Socket, J3 4P4C, J4 OLED_128x32, J5 Conn_01x02_Socket, J6 4P4C, SW1 Switch, SW2 SW_SPDT, SW3 Switch, SW4 SW_SPDT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

Commit message: reroute for full duplex split functionality
Connections:
- J3 pad 3: L_SCL -> L_TX
- J3 pad 4: L_SDA -> L_RX
- J6 pad 3: R_SCL -> R_RX
- J6 pad 4: R_SDA -> R_TX
- U1 pad 7: unconnected-(U1-U0TXD_D6/TX-Pad7) -> L_TX
- U1 pad 8: unconnected-(U1-U0RXD_D7/RX-Pad8)_1 -> L_RX
- U3 pad 7: unconnected-(U3-U0TXD_D6/TX-Pad7)_1 -> R_TX
- U3 pad 8: unconnected-(U3-U0RXD_D7/RX-Pad8) -> R_RX
Routing:
- net L_TX: track 0.00 -> 48.3 mm
- net R_RX: track 0.00 -> 45.6 mm
- net GND: track 157.7 -> 181.4 mm
- net R_SDA: track 37.5 -> 20.0 mm
- net R_TX: track 0.00 -> 16.8 mm
- net R_SCL: track 31.7 -> 15.3 mm
- net L_SCL: track 35.7 -> 19.5 mm
- net R_RAW: track 72.8 -> 61.3 mm
- net L_RX: track 0.00 -> 10.2 mm
- net L_SDA: track 34.0 -> 28.5 mm
- net +5V: track 52.2 -> 54.1 mm
- net R_COL1: track 202.2 -> 200.9 mm
- net unconnected-(U3-U0TXD_D6/TX-Pad7)_1: track 1.27 -> 0.00 mm
- net unconnected-(U3-U0RXD_D7/RX-Pad8): track 1.27 -> 0.00 mm
- net unconnected-(U3-GPIO4_D3/A3-Pad4)_1: track 1.27 -> 0.00 mm
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Other:
- board text added: "JLCJLCJLCJLC"
