File: CAD/KiCad/keyboard.kicad_sch (KiCad schematic)
At the start: 120 parts, among them J1 OLED_128x32, J2 Conn_01x02_Socket, J3 4P4C, J4 OLED_128x32, J5 Conn_01x02_Socket, J6 4P4C, SW1 Switch, SW2 SW_SPDT, SW3 Switch, SW4 SW_SPDT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

Commit message: reroute for full duplex split functionality
Connections:
- net L_SCL: no longer J3.3
- net L_SDA: no longer J3.4
- net R_SCL: no longer J6.3
- net R_SDA: no longer J6.4
- net R_TX: now reaches U3.7 (U0TXD_D6/TX)
- net R_TX: now also J6.4
- net R_RX: now reaches U3.8 (U0RXD_D7/RX)
- net R_RX: now also J6.3
- net L_TX: now reaches U1.7 (U0TXD_D6/TX)
- net L_TX: now also J3.3
- net L_RX: now reaches U1.8 (U0RXD_D7/RX)
- net L_RX: now also J3.4
- no-connect marks 28 -> 24
